File: hardware/rev0/amalthea_rev0.sch (KiCad schematic (older format))
At the start: 34 parts, among them J1 USB_B_Micro, J2 USB_B_Micro, J3 USB_A, J4 USB_B_Micro, J7 Conn_02x02_Counter_Clockwise, J8 Conn_Coaxial, J9 Conn_Coaxial, SW1 BTN_RECOVERY, SW2 BTN_DFU, SW3 BTN_RESET, U1 AP22814-SOT, U12 AP22814-SOT, Y1 DSC60xx

Commit message: Bulk rename
Parts:
- D1, D8: footprint luna:SOD128 -> amalthea:SOD128
- J3: footprint luna:CONN-Amphenol-UE27AC54100 -> amalthea:CONN-Amphenol-UE27AC54100
- J8, J9: footprint luna:SMA-EDGE -> amalthea:SMA-EDGE
- SW1, SW2, SW3: footprint luna:SWITCH-FSMRA -> amalthea:SWITCH-FSMRA
Changed lines of the file:
@@
 EESchema Schematic File Version 4
-LIBS:luna_rev0-cache
+LIBS:amalthea_rev0-cache
 EELAYER 29 0
 EELAYER END
@@
 encoding utf-8
 Sheet 1 9
-Title "LUNA USB Multitool"
+Title "Amalthea USB Multitool"
 Date "2019-10-20"
 Rev "r0"
@@
 F 0 "D8" H 6300 4950 50  0000 C CNN
 F 1 "PMEG3050EP,115" H 6200 5000 50  0001 C CNN
-F 2 "luna:SOD128" H 6300 4850 50  0001 C CNN
+F 2 "amalthea:SOD128" H 6300 4850 50  0001 C CNN
 F 3 "~" H 6300 4850 50  0001 C CNN
 	1    6300 4850
@@
 F 0 "D1" H 1500 3650 50  0000 C CNN
 F 1 "PMEG3050EP,115" H 1400 3700 50  0001 C CNN
-F 2 "luna:SOD128" H 1500 3550 50  0001 C CNN
+F 2 "amalthea:SOD128" H 1500 3550 50  0001 C CNN
 F 3 "~" H 1500 3550 50  0001 C CNN
 	1    1500 3550
@@
 F 0 "J3" H 8721 2439 50  0000 R CNN
 F 1 "USB_A" H 8721 2349 50  0000 R CNN
-F 2 "luna:CONN-Amphenol-UE27AC54100" H 9100 2400 50  0001 C CNN
+F 2 "amalthea:CONN-Amphenol-UE27AC54100" H 9100 2400 50  0001 C CNN
 F 3 " ~" H 9100 2400 50  0001 C CNN
 	1    8950 2450
@@
 F 0 "SW1" H 2000 5400 50  0000 C CNN
 F 1 "BTN_RECOVERY" H 2250 5250 50  0000 C CNN
-F 2 "luna:SWITCH-FSMRA" H 2250 5350 50  0001 C CNN
+F 2 "amalthea:SWITCH-FSMRA" H 2250 5350 50  0001 C CNN
 F 3 "~" H 2250 5350 50  0001 C CNN
 	1    2250 5350
@@
 F 0 "SW2" H 2000 5700 50  0000 C CNN
 F 1 "BTN_DFU" H 2250 5500 50  0000 C CNN
-F 2 "luna:SWITCH-FSMRA" H 2250 5650 50  0001 C CNN
+F 2 "amalthea:SWITCH-FSMRA" H 2250 5650 50  0001 C CNN
 F 3 "~" H 2250 5650 50  0001 C CNN
 	1    2250 5650
@@
 F 0 "SW3" H 2000 6050 50  0000 C CNN
 F 1 "BTN_RESET" H 2250 5900 50  0000 C CNN
-F 2 "luna:SWITCH-FSMRA" H 2250 6000 50  0001 C CNN
+F 2 "amalthea:SWITCH-FSMRA" H 2250 6000 50  0001 C CNN
 F 3 "~" H 2250 6000 50  0001 C CNN
 	1    2250 6000
@@
 F 0 "J8" H 3450 974 50  0000 L CNN
 F 1 "Conn_Coaxial" H 3450 884 50  0001 L CNN
-F 2 "luna:SMA-EDGE" H 3350 1000 50  0001 C CNN
+F 2 "amalthea:SMA-EDGE" H 3350 1000 50  0001 C CNN
 F 3 " ~" H 3350 1000 50  0001 C CNN
 	1    3350 1000
@@
 F 0 "J9" H 3449 1329 50  0000 L CNN
 F 1 "Conn_Coaxial" H 3450 1284 50  0001 L CNN
-F 2 "luna:SMA-EDGE" H 3350 1400 50  0001 C CNN
+F 2 "amalthea:SMA-EDGE" H 3350 1400 50  0001 C CNN
 F 3 " ~" H 3350 1400 50  0001 C CNN
 	1    3350 1400
