File: hardware/rev0/host_side.sch (KiCad schematic (older format))
At the start: 9 parts, among them IC1 ECP5-BGA256, U11 USB3343

Commit message: Bulk rename
Parts:
- IC1: footprint luna:lattice_cabga256 -> amalthea:lattice_cabga256
Changed lines of the file:
@@
 EESchema Schematic File Version 4
-LIBS:luna_rev0-cache
+LIBS:amalthea_rev0-cache
 EELAYER 29 0
 EELAYER END
@@
 encoding utf-8
 Sheet 7 9
-Title "LUNA: Upstream \"Host\" Section"
+Title "Amalthea: Upstream \"Host\" Section"
 Date "2019-10-20"
 Rev "r0"
@@
 F 0 "IC1" H 1670 -617 50  0000 R CNN
 F 1 "ECP5-BGA256" H 1670 -707 50  0000 R CNN
-F 2 "luna:lattice_cabga256" H -1500 4950 50  0001 L CNN
+F 2 "amalthea:lattice_cabga256" H -1500 4950 50  0001 L CNN
 F 3 "" H -1950 5900 50  0001 L CNN
 F 4 "FPGA - Field Programmable Gate Array ECP5; 12k LUTs; 1.1V" H -1950 5800 50  0001 L CNN "Description"
