File: hardware/rev0/power_supplies.sch (KiCad schematic (older format))
At the start: 40 parts, among them IC1 ECP5-BGA256, U2 MIC5504-1.8YM5, U3 MIC5219-3.3YM5, U4 TCR2EF11, U5 MIC5504-2.5YM5

Commit message: Bulk rename
Parts:
- IC1: footprint luna:lattice_cabga256 -> amalthea:lattice_cabga256
Changed lines of the file:
@@
 EESchema Schematic File Version 4
-LIBS:luna_rev0-cache
+LIBS:amalthea_rev0-cache
 EELAYER 29 0
 EELAYER END
@@
 encoding utf-8
 Sheet 2 9
-Title "LUNA: Power Supplies"
+Title "Amalthea: Power Supplies"
 Date "2019-10-20"
 Rev "r0"
@@
 F 0 "IC1" H 9100 3368 50  0000 C CNN
 F 1 "ECP5-BGA256" H 9100 3277 50  0000 C CNN
-F 2 "luna:lattice_cabga256" H 5150 6650 50  0001 L CNN
+F 2 "amalthea:lattice_cabga256" H 5150 6650 50  0001 L CNN
 F 3 "" H 4700 7600 50  0001 L CNN
 F 4 "FPGA - Field Programmable Gate Array ECP5; 12k LUTs; 1.1V" H 4700 7500 50  0001 L CNN "Description"
