File: hardware/rev0/ram_section.sch (KiCad schematic (older format))
At the start: 2 parts, among them IC1 ECP5-BGA256, U10 S27KS0641

Commit message: Bulk rename
Parts:
- IC1: footprint luna:lattice_cabga256 -> amalthea:lattice_cabga256
- U10: footprint luna:BGA-24_5x5_6.0x8.0mm -> amalthea:BGA-24_5x5_6.0x8.0mm
Changed lines of the file:
@@
 EESchema Schematic File Version 4
-LIBS:luna_rev0-cache
+LIBS:amalthea_rev0-cache
 EELAYER 29 0
 EELAYER END
@@
 encoding utf-8
 Sheet 6 9
-Title "LUNA: RAM Section"
+Title "Amalthea: RAM Section"
 Date "2019-10-20"
 Rev "r0"
@@
 F 0 "IC1" H 1620 308 50  0000 R CNN
 F 1 "ECP5-BGA256" H 1620 218 50  0000 R CNN
-F 2 "luna:lattice_cabga256" H -1550 5550 50  0001 L CNN
+F 2 "amalthea:lattice_cabga256" H -1550 5550 50  0001 L CNN
 F 3 "" H -2000 6500 50  0001 L CNN
 F 4 "FPGA - Field Programmable Gate Array ECP5; 12k LUTs; 1.1V" H -2000 6400 50  0001 L CNN "Description"
@@
 F 0 "U10" H 5400 5772 50  0000 C CNN
 F 1 "S27KS0641" H 5400 5682 50  0000 C CNN
-F 2 "luna:BGA-24_5x5_6.0x8.0mm" H 6000 3950 50  0001 C CNN
+F 2 "amalthea:BGA-24_5x5_6.0x8.0mm" H 6000 3950 50  0001 C CNN
 F 3 "" H 5400 3950 50  0001 C CNN
 F 4 "ANY" H 5400 4850 50  0001 C CNN "Source"
