File: hardware/rev0/right_side_indicators.sch (KiCad schematic (older format))
At the start: 1 part, among them IC1 ECP5-BGA256

Commit message: Bulk rename
Parts:
- IC1: footprint luna:lattice_cabga256 -> amalthea:lattice_cabga256
Changed lines of the file:
@@
 EESchema Schematic File Version 4
-LIBS:luna_rev0-cache
+LIBS:amalthea_rev0-cache
 EELAYER 29 0
 EELAYER END
@@
 encoding utf-8
 Sheet 9 9
-Title "LUNA: Right Side I/O"
+Title "Amalthea: Right Side I/O"
 Date "2019-10-20"
 Rev "r0"
@@
 F 0 "IC1" H 2120 208 50  0000 R CNN
 F 1 "ECP5-BGA256" H 2120 118 50  0000 R CNN
-F 2 "luna:lattice_cabga256" H -1050 5450 50  0001 L CNN
+F 2 "amalthea:lattice_cabga256" H -1050 5450 50  0001 L CNN
 F 3 "" H -1500 6400 50  0001 L CNN
 F 4 "FPGA - Field Programmable Gate Array ECP5; 12k LUTs; 1.1V" H -1500 6300 50  0001 L CNN "Description"
