File: hardware/rev0/target_side.sch (KiCad schematic (older format))
At the start: 9 parts, among them IC1 ECP5-BGA256, U9 USB3343

Commit message: Bulk rename
Parts:
- IC1: footprint luna:lattice_cabga256 -> amalthea:lattice_cabga256
Changed lines of the file:
@@
 EESchema Schematic File Version 4
-LIBS:luna_rev0-cache
+LIBS:amalthea_rev0-cache
 EELAYER 29 0
 EELAYER END
@@
 encoding utf-8
 Sheet 5 9
-Title "LUNA: Downstream / Target / Analysis Section"
+Title "Amalthea: Downstream / Target / Analysis Section"
 Date "2019-10-20"
 Rev "r0"
@@
 F 0 "IC1" H 1620 283 50  0000 R CNN
 F 1 "ECP5-BGA256" H 1620 193 50  0000 R CNN
-F 2 "luna:lattice_cabga256" H -1550 5550 50  0001 L CNN
+F 2 "amalthea:lattice_cabga256" H -1550 5550 50  0001 L CNN
 F 3 "" H -2000 6500 50  0001 L CNN
 F 4 "FPGA - Field Programmable Gate Array ECP5; 12k LUTs; 1.1V" H -2000 6400 50  0001 L CNN "Description"
