File: hardware/rev0/target_side.sch (KiCad schematic (older format))
At the start: 31 parts, among them IC1 ECP5-BGA256, U1 2450FB15A050, U12 0896BM15E0025, U13 TXETALSANF-26.000000, U9 AT86RF215

Commit message: Pick part numbers for BOM
Parts:
- C40, C41, C59: Manufacturer_Part_Number (none) -> LMK105BJ105KPLF
- C42, C46: value 1.8pF -> 1.8pF RF; Manufacturer_Part_Number (none) -> 04021J1R8BBSTR
- C43: value 0.8pF -> 0.8pF RF; Manufacturer_Part_Number (none) -> 04023J0R8BBSTR
- C53: value 15pF -> 15pF RF; Manufacturer_Part_Number (none) -> 04023K150FBSTR
- C56: Manufacturer_Part_Number (none) -> TMF105B7102KVHF
- C57, C60, C61, C62, C63, C64: Manufacturer_Part_Number (none) -> LMF105B7104KVHF
- C58: Manufacturer_Part_Number (none) -> C0402C100K5RACTU
- L1: value 5.6nH -> 5.6nH RF; Manufacturer_Part_Number (none) -> MLG1005S5N6CT000
- R1, R3: Manufacturer_Part_Number (none) -> CRCW04020000Z0ED
- R2, R4, R5: Manufacturer_Part_Number (none) -> CRCW040210K0FKEDC
- R6: Manufacturer_Part_Number (none) -> CRCW0402100KFKEDC
- U1: Manufacturer_Part_Number (none) -> 2450FB15A050
- U12: Manufacturer_Part_Number (none) -> 0896BM15E0025
- U13: Manufacturer_Part_Number (none) -> ECS-TXO-32CSMV-260-AN-TR
- U9: Manufacturer_Part_Number (none) -> 556-AT86RF215IQ-ZUR
Changed lines of the file:
@@
 F 2 "Package_DFN_QFN:QFN-48-1EP_7x7mm_P0.5mm_EP5.6x5.6mm" H 5150 3650 50  0001 C CNN
 F 3 "" H 5150 3650 50  0001 C CNN
+F 4 "556-AT86RF215IQ-ZUR" H 5150 3900 50  0001 C CNN "Manufacturer_Part_Number"
 	1    5150 3900
 	1    0    0    -1
@@
 F 2 "Capacitor_SMD:C_0402_1005Metric" H 6038 4850 50  0001 C CNN
 F 3 "~" H 6000 5000 50  0001 C CNN
+F 4 "LMK105BJ105KPLF" H 6000 5000 50  0001 C CNN "Manufacturer_Part_Number"
 	1    6000 5000
 	1    0    0    -1
@@
 F 2 "Capacitor_SMD:C_0402_1005Metric" H 6438 4850 50  0001 C CNN
 F 3 "~" H 6400 5000 50  0001 C CNN
+F 4 "LMK105BJ105KPLF" H 6400 5000 50  0001 C CNN "Manufacturer_Part_Number"
 	1    6400 5000
 	1    0    0    -1
@@
 F 2 "amalthea:Filter_Johanson_2x1.25mm" H 8350 3750 50  0001 C CNN
 F 3 "" H 8350 3750 50  0001 C CNN
+F 4 "2450FB15A050" H 8350 3200 50  0001 C CNN "Manufacturer_Part_Number"
 	1    8350 3200
 	1    0    0    -1
@@
 F 2 "amalthea:Filter_Johanson_2x1.25mm" H 8350 4800 50  0001 C CNN
 F 3 "" H 8350 4800 50  0001 C CNN
+F 4 "0896BM15E0025" H 8350 4400 50  0001 C CNN "Manufacturer_Part_Number"
 	1    8350 4400
 	1    0    0    -1
@@
 P 7250 2750
 F 0 "C42" V 6998 2750 50  0000 C CNN
-F 1 "1.8pF" V 7089 2750 50  0000 C CNN
+F 1 "1.8pF RF" V 7089 2750 50  0000 C CNN
 F 2 "Capacitor_SMD:C_0402_1005Metric" H 7288 2600 50  0001 C CNN
 F 3 "~" H 7250 2750 50  0001 C CNN
+F 4 "04021J1R8BBSTR" H 7250 2750 50  0001 C CNN "Manufacturer_Part_Number"
 	1    7250 2750
 	0    1    1    0
@@
 P 7250 3250
 F 0 "C46" V 7502 3250 50  0000 C CNN
-F 1 "1.8pF" V 7411 3250 50  0000 C CNN
+F 1 "1.8pF RF" V 7411 3250 50  0000 C CNN
 F 2 "Capacitor_SMD:C_0402_1005Metric" H 7288 3100 50  0001 C CNN
 F 3 "~" H 7250 3250 50  0001 C CNN
+F 4 "04021J1R8BBSTR" H 7250 3250 50  0001 C CNN "Manufacturer_Part_Number"
 	1    7250 3250
 	0    -1   -1   0
@@
 P 7500 3000
 F 0 "L1" H 7553 3046 50  0000 L CNN
-F 1 "5.6nH" H 7553 2955 50  0000 L CNN
+F 1 "5.6nH RF" H 7553 2955 50  0000 L CNN
 F 2 "Inductor_SMD:L_0402_1005Metric" H 7500 3000 50  0001 C CNN
 F 3 "~" H 7500 3000 50  0001 C CNN
+F 4 "MLG1005S5N6CT000" H 7500 3000 50  0001 C CNN "Manufacturer_Part_Number"
 	1    7500 3000
 	1    0    0    -1
@@
 P 8950 2950
 F 0 "C43" V 8698 2950 50  0000 C CNN
-F 1 "0.8pF" V 8789 2950 50  0000 C CNN
+F 1 "0.8pF RF" V 8789 2950 50  0000 C CNN
 F 2 "Capacitor_SMD:C_0402_1005Metric" H 8988 2800 50  0001 C CNN
 F 3 "~" H 8950 2950 50  0001 C CNN
+F 4 "04023J0R8BBSTR" H 8950 2950 50  0001 C CNN "Manufacturer_Part_Number"
 	1    8950 2950
 	0    1    1    0
@@
 F 2 "Resistor_SMD:R_0402_1005Metric" V 9380 2950 50  0001 C CNN
 F 3 "~" H 9450 2950 50  0001 C CNN
+F 4 "CRCW04020000Z0ED" H 9450 2950 50  0001 C CNN "Manufacturer_Part_Number"
 	1    9450 2950
 	0    1    1    0
@@
 F 2 "Resistor_SMD:R_0402_1005Metric" V 10130 3200 50  0001 C CNN
 F 3 "~" H 10200 3200 50  0001 C CNN
+F 4 "CRCW040210K0FKEDC" H 10200 3200 50  0001 C CNN "Manufacturer_Part_Number"
 	1    10200 3200
 	-1   0    0    1
@@
 P 8950 4300
 F 0 "C53" V 8698 4300 50  0000 C CNN
-F 1 "15pF" V 8789 4300 50  0000 C CNN
+F 1 "15pF RF" V 8789 4300 50  0000 C CNN
 F 2 "Capacitor_SMD:C_0402_1005Metric" H 8988 4150 50  0001 C CNN
 F 3 "~" H 8950 4300 50  0001 C CNN
+F 4 "04023K150FBSTR" H 8950 4300 50  0001 C CNN "Manufacturer_Part_Number"
 	1    8950 4300
 	0    1    1    0
@@
 F 2 "Resistor_SMD:R_0402_1005Metric" V 9380 4300 50  0001 C CNN
 F 3 "~" H 9450 4300 50  0001 C CNN
+F 4 "CRCW04020000Z0ED" H 9450 4300 50  0001 C CNN "Manufacturer_Part_Number"
 	1    9450 4300
 	0    1    1    0
@@
 F 2 "Resistor_SMD:R_0402_1005Metric" V 10130 4550 50  0001 C CNN
 F 3 "~" H 10200 4550 50  0001 C CNN
+F 4 "CRCW040210K0FKEDC" H 10200 4550 50  0001 C CNN "Manufacturer_Part_Number"
 	1    10200 4550
 	-1   0    0    1
@@
 F 2 "Oscillator:Oscillator_SMD_SeikoEpson_SG8002CE-4Pin_3.2x2.5mm" H 2450 1850 50  0001 C CNN
 F 3 "" H 2450 1850 50  0001 C CNN
+F 4 "ECS-TXO-32CSMV-260-AN-TR" H 2400 1350 50  0001 C CNN "Manufacturer_Part_Number"
 	1    2400 1350
 	1    0    0    -1
@@
 F 2 "Capacitor_SMD:C_0402_1005Metric" H 1538 1300 50  0001 C CNN
 F 3 "~" H 1500 1450 50  0001 C CNN
+F 4 "LMF105B7104KVHF" H 1500 1450 50  0001 C CNN "Manufacturer_Part_Number"
 	1    1500 1450
 	1    0    0    -1
@@
 F 2 "Capacitor_SMD:C_0402_1005Metric" H 3138 1200 50  0001 C CNN
 F 3 "~" H 3100 1350 50  0001 C CNN
+F 4 "TMF105B7102KVHF" H 3100 1350 50  0001 C CNN "Manufacturer_Part_Number"
 	1    3100 1350
 	0    1    1    0
@@
 F 2 "Resistor_SMD:R_0402_1005Metric" V 3280 1550 50  0001 C CNN
 F 3 "~" H 3350 1550 50  0001 C CNN
+F 4 "CRCW040210K0FKEDC" H 3350 1550 50  0001 C CNN "Manufacturer_Part_Number"
 	1    3350 1550
 	1    0    0    -1
@@
 F 2 "Capacitor_SMD:C_0402_1005Metric" H 3738 1400 50  0001 C CNN
 F 3 "~" H 3700 1550 50  0001 C CNN
+F 4 "C0402C100K5RACTU" H 3700 1550 50  0001 C CNN "Manufacturer_Part_Number"
 	1    3700 1550
 	1    0    0    -1
@@
 F 2 "Resistor_SMD:R_0402_1005Metric" V 4030 3050 50  0001 C CNN
 F 3 "~" H 4100 3050 50  0001 C CNN
+F 4 "CRCW0402100KFKEDC" H 4100 3050 50  0001 C CNN "Manufacturer_Part_Number"
 	1    4100 3050
 	0    1    1    0
@@
 F 2 "Capacitor_SMD:C_0402_1005Metric" H 6838 4850 50  0001 C CNN
 F 3 "~" H 6800 5000 50  0001 C CNN
+F 4 "LMK105BJ105KPLF" H 6800 5000 50  0001 C CNN "Manufacturer_Part_Number"
 	1    6800 5000
 	1    0    0    -1
@@
 F 2 "Capacitor_SMD:C_0402_1005Metric" H 4238 6650 50  0001 C CNN
 F 3 "~" H 4200 6800 50  0001 C CNN
+F 4 "LMF105B7104KVHF" H 4200 6800 50  0001 C CNN "Manufacturer_Part_Number"
 	1    4200 6800
 	1    0    0    -1
@@
 F 2 "Capacitor_SMD:C_0402_1005Metric" H 4738 6650 50  0001 C CNN
 F 3 "~" H 4700 6800 50  0001 C CNN
+F 4 "LMF105B7104KVHF" H 4700 6800 50  0001 C CNN "Manufacturer_Part_Number"
 	1    4700 6800
 	1    0    0    -1
@@
 F 2 "Capacitor_SMD:C_0402_1005Metric" H 5238 6650 50  0001 C CNN
 F 3 "~" H 5200 6800 50  0001 C CNN
+F 4 "LMF105B7104KVHF" H 5200 6800 50  0001 C CNN "Manufacturer_Part_Number"
 	1    5200 6800
 	1    0    0    -1
@@
 F 2 "Capacitor_SMD:C_0402_1005Metric" H 5738 6650 50  0001 C CNN
 F 3 "~" H 5700 6800 50  0001 C CNN
+F 4 "LMF105B7104KVHF" H 5700 6800 50  0001 C CNN "Manufacturer_Part_Number"
 	1    5700 6800
 	1    0    0    -1
@@
 F 2 "Capacitor_SMD:C_0402_1005Metric" H 6238 6650 50  0001 C CNN
 F 3 "~" H 6200 6800 50  0001 C CNN
+F 4 "LMF105B7104KVHF" H 6200 6800 50  0001 C CNN "Manufacturer_Part_Number"
 	1    6200 6800
 	1    0    0    -1
